File: Blast Furnace PCB.kicad_pcb (KiCad board)
At the start: 2 copper layers, 84 x 60 mm, 35 parts, among them J1 Thermocouple_Screw_Terminal_0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, J2 9V_Conn_01x02, J3 Conn_02x06_Odd_Even, Q1 BSS138, Q2 BSS138, SW1 POWER_SWITCH, U1 MAX31856, U2 I2C_16x2_LCD

Commit message: standard save stuff
Other:
- board text added: "Blast Furnace Temperature Sensor Display V1.2.3 (Inhouse Version)"
- board text removed: "Blast Furnace Temperature Sensor Display V1.2 (Inhouse Version)"
